Commit message: i

File: murin_bringup/description/2wd/robot_core.2wd.xacro (robot description, xacro)
@@ -1,6 +1,6 @@
 <?xml version="1.0"?>
 <robot xmlns:xacro="http://www.ros.org/wiki/xacro">
-    <xacro:include filename="$(find murin_bringup)/desciption/macros/inertial_macros.xacro" />
-    <xacro:include filename="$(find murin_bringup)/desciption/macros/wheel.macros.xacro"/>
+    <xacro:include filename="$(find murin_bringup)/description/macros/inertial_macros.xacro" />
+    <xacro:include filename="$(find murin_bringup)/description/macros/wheel.macros.xacro"/>
     <xacro:property name="chassis_length" value="0.225"/>
     <xacro:property name="chassis_width" value="0.153"/>

File: murin_bringup/description/4wd/robot_core.4wd.xacro (robot description, xacro)
@@ -1,6 +1,6 @@
 <?xml version="1.0"?>
 <robot xmlns:xacro="http://www.ros.org/wiki/xacro">
-    <xacro:include filename="$(find murin_bringup)/desciption/macros/inertial_macros.xacro" />
-    <xacro:include filename="$(find murin_bringup)/desciption/macros/wheel.macros.xacro"/>
+    <xacro:include filename="$(find murin_bringup)/description/macros/inertial_macros.xacro" />
+    <xacro:include filename="$(find murin_bringup)/description/macros/wheel.macros.xacro"/>
     <xacro:property name="chassis_length" value="0.225"/>
     <xacro:property name="chassis_width" value="0.153"/>

File: murin_bringup/description/accessories/dept_camera.xacro (robot description, xacro)
@@ -25,5 +25,5 @@
         <parent link="base_link"/>
         <child link="camera_link"/>
-        <origin xyz="0.1125 0.0 0.03" rpy="0 0 0"/>
+        <origin xyz="0.110 0.0 0.111" rpy="0 0 0"/>
     </joint>
     <!-- Camera depth link -->

File: murin_bringup/description/robot.urdf.xacro (robot description, xacro)
@@ -3,7 +3,7 @@
     <xacro:include filename="4wd/robot_core.4wd.xacro" />
     <xacro:include filename="ros2_control.xacro" />
-    <!-- <xacro:include filename="accessories/lidar.xacro" /> -->
+    <xacro:include filename="accessories/lidar.xacro" />
     <!-- <xacro:include filename="accessories/camera.xacro" /> -->
-    <!-- <xacro:include filename="accessories/dept_camera.xacro" /> -->
-    <!-- <xacro:include filename="accessories/imu.xacro" /> -->
+    <xacro:include filename="accessories/dept_camera.xacro" />
+    <xacro:include filename="accessories/imu.xacro" />
 </robot>

File: murin_bringup/description/ros2_control.xacro (robot description, xacro)
@@ -3,5 +3,5 @@
     <ros2_control name="DiffBot" type="system">
         <hardware>
-            <plugin>diffdrive_arduino/DiffDriveArduinoHardware</plugin>
+            <plugin>murin_base/MurinBaseHardware</plugin>
             <param name="front_left_wheel_name">front_left_wheel_joint</param>
             <param name="rear_left_wheel_name">rear_left_wheel_joint</param>
@@ -38,4 +38,16 @@
             <state_interface name="velocity"/>
         </joint>
+        <sensor name='mpu6050'>
+        <state_interface name='orientation.x'/>
+        <state_interface name='orientation.y'/>
+        <state_interface name='orientation.z'/>
+        <state_interface name='orientation.w'/>
+        <state_interface name='angular_velocity.x'/>
+        <state_interface name='angular_velocity.y'/>
+        <state_interface name='angular_velocity.z'/>
+        <state_interface name='linear_acceleration.x'/>
+        <state_interface name='linear_acceleration.y'/>
+        <state_interface name='linear_acceleration.z'/>
+      </sensor>
     </ros2_control>
 </robot>
