Commit message: i

File: murin_bringup/description/4wd/robot_core.4wd.xacro (robot description, xacro)
@@ -46,12 +46,13 @@
         <parent link="base_link"/>
         <child link="chassis"/>
-        <origin xyz="0 0 ${-chassis_offset_z}"/>
+        <origin xyz="0 0 0"/>
     </joint>
     <link name="chassis">
         <!-- chassis visual -->
         <visual>
-            <origin xyz="0 0 ${chassis_height/2}"/>
+            <origin xyz="0 0 0"/>
             <geometry>
-                <box size="${chassis_length} ${chassis_width} ${chassis_height}"/>
+                <mesh filename="package://murin_bringup/description/meshes/base_link.STL" />
+                <!-- <box size="${chassis_length} ${chassis_width} ${chassis_height}"/> -->
             </geometry>
             <material name="white"/>

File: murin_bringup/description/accessories/dept_camera.xacro (robot description, xacro)
@@ -6,5 +6,6 @@
             <origin xyz="0 0 0" rpy="0 0 0"/>
             <geometry>
-            <box size="0.025 0.095 0.025"/>
+                <mesh filename="package://murin_bringup/description/meshes/camera_link.STL" />
+                <!-- <box size="0.025 0.095 0.025"/> -->
             </geometry>
         </visual>

File: murin_bringup/description/accessories/lidar.xacro (robot description, xacro)
@@ -17,5 +17,6 @@
             <origin xyz="0 0 0" rpy="0 0 0"/>
             <geometry>
-                <cylinder radius="0.017" length="0.014"/>
+                <mesh filename="package://murin_bringup/description/meshes/lidar_link.STL" />
+                <!-- <cylinder radius="0.017" length="0.014"/> -->
             </geometry>
         </visual>

File: murin_bringup/description/macros/wheel.macros.xacro (robot description, xacro)
@@ -5,7 +5,8 @@
         <link name="${prefix}_wheel">
             <visual>
-                <origin xyz="0 0 0" rpy="${pi/2} 0 0" />
+                <origin xyz="0 0 0" rpy="0 0 0" />
                 <geometry>
-                    <cylinder radius="${wheel_radius}" length="${wheel_length}"/>
+                    <mesh filename="package://murin_bringup/description/meshes/${prefix}_wheel.STL" />
+                    <!-- <cylinder radius="${wheel_radius}" length="${wheel_length}"/> -->
                 </geometry>
                 <material name="blue"/>
