Commit message: i

File: murin_bringup/description/accessories/lidar.xacro (robot description, xacro)
@@ -64,10 +64,10 @@
         </sensor>
     </gazebo>
-    <joint name="laser_joint" type="fixed">
+    <!-- <joint name="laser_joint" type="fixed">
         <parent link="base_link"/>
         <child link="laser_frame"/>
         <origin xyz="0.074 -0.04 0.0775" rpy="0.0 0.0 0.0"/>
-    </joint>
-    <link name="laser_frame">
+    </joint> -->
+    <!-- <link name="laser_frame">
         <visual>
             <origin xyz="0 0 0.007" rpy="0 0 0"/>
@@ -114,4 +114,4 @@
             </plugin>
         </sensor>
-    </gazebo>
+    </gazebo> -->
 </robot>
