Commit message: i

File: murin_base/description/ros2_control/diffbot.ros2_control.xacro (robot description, xacro)
@@ -11,5 +11,6 @@
         <param name="loop_rate">50</param>
         <!-- <param name="device">/dev/agv-driver</param> -->
-        <param name="device">/dev/ldlidar</param>
+        <param name="robot_driver">/dev/robot_driver</param>
+        <param name="robot_imu">/dev/robot_imu</param>
         <param name="baud_rate">460800</param>
         <param name="timeout_ms">1000</param>

File: murin_base/description/urdf/diffbot_description.urdf.xacro (robot description, xacro)
@@ -51,11 +51,11 @@
     <joint name="${prefix}rear_left_wheel_joint" type="continuous">
       <parent link="${prefix}base_link"/>
-      <child link="${prefix}left_wheel"/>
-      <origin xyz="-${wheel_offset_x} -${wheel_offset_y} 0" rpy="0 0 0"/>
+      <child link="${prefix}rear_left_wheel"/>
+      <origin xyz="-${wheel_offset_x} ${wheel_offset_y} 0" rpy="0 0 0"/>
       <axis xyz="0 1 0"/>
       <dynamics damping="0.2"/>
     </joint>
     <!-- left wheel Link -->
-    <link name="${prefix}left_wheel">
+    <link name="${prefix}rear_left_wheel">
       <collision>
         <origin xyz="0 0 0" rpy="${PI/2} 0 0"/>
@@ -83,5 +83,5 @@
       <parent link="${prefix}base_link"/>
       <child link="${prefix}front_left_wheel"/>
-      <origin xyz="${wheel_offset_x} -${wheel_offset_y} 0" rpy="0 0 0"/>
+      <origin xyz="${wheel_offset_x} ${wheel_offset_y} 0" rpy="0 0 0"/>
       <axis xyz="0 1 0"/>
       <dynamics damping="0.2"/>
@@ -113,11 +113,11 @@
     <joint name="${prefix}rear_right_wheel_joint" type="continuous">
       <parent link="${prefix}base_link"/>
-      <child link="${prefix}right_wheel"/>
-      <origin xyz="-${wheel_offset_x} ${wheel_offset_y} 0" rpy="0 0 0"/>
+      <child link="${prefix}rear_right_wheel"/>
+      <origin xyz="-${wheel_offset_x} -${wheel_offset_y} 0" rpy="0 0 0"/>
       <axis xyz="0 1 0"/>
       <dynamics damping="0.2"/>
     </joint>
     <!-- right wheel Link -->
-    <link name="${prefix}right_wheel">
+    <link name="${prefix}rear_right_wheel">
       <collision>
         <origin xyz="0 0 0" rpy="${PI/2} 0 0"/>
@@ -145,5 +145,5 @@
       <parent link="${prefix}base_link"/>
       <child link="${prefix}front_right_wheel"/>
-      <origin xyz="${wheel_offset_x} ${wheel_offset_y} 0" rpy="0 0 0"/>
+      <origin xyz="${wheel_offset_x} -${wheel_offset_y} 0" rpy="0 0 0"/>
       <axis xyz="0 1 0"/>
       <dynamics damping="0.2"/>

File: murin_bringup/description/ros2_control.xacro (robot description, xacro)
@@ -8,6 +8,7 @@
             <param name="front_right_wheel_name">front_right_wheel_joint</param>
             <param name="rear_right_wheel_name">rear_right_wheel_joint</param>
-            <param name="loop_rate">30</param>
-            <param name="device">/dev/agv-driver</param>
+            <param name="loop_rate">50</param>
+            <param name="robot_driver">/dev/robot_driver</param>
+            <param name="robot_imu">/dev/robot_imu</param>
             <param name="baud_rate">460800</param>
             <param name="timeout_ms">1000</param>
